Commit message: v1 design

File: jetbot_description/urdf/jetbot_description.urdf (robot description, URDF)
Before this commit: robot jetbot_description, 5 links, 4 joints
Links:
- removed link intel_d435
- removed link left_wheel
- removed link right_wheel
- added link camera, mass 1.2669; collision mesh filename=package://jetbot_description/meshes/camera.STL; visual mesh filename=package://jetbot_description/meshes/camera.STL
- link base_link: mass 0.769809092579164 -> 0.89553
- link laser: mass 0.0730824507861898 -> 0.073082; geometry collision mesh filename=package://jetbot_description/meshes/laser.STL; visual mesh filename=package://jetbot_description/meshes/laser.STL
Joints:
- removed joint joint_lw
- removed joint joint_rw
- joint joint_camera: child intel_d435 -> camera; origin xyz=0.027 0 0.1175 rpy=1.5708 0 1.5708 -> xyz=0.020034 0 0.14645 rpy=1.5708 0 1.5708
- joint joint_laser: origin xyz=-0.1325 0.015 0.1485 rpy=0 0 -1.5708 -> xyz=-0.071 0 0.176 rpy=0 0 3.1416
